File: hardware/slimsata-2.brd (EAGLE design)
At the start: 20.3 x 64.8 mm, 2 parts

Commit message: Masse nochmal neu
Routing:
- net GND: track 198.4 -> 255.7 mm, vias 24 -> 25
Changed lines of the file:
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@@
 <wire x1="5.386" y1="30.532" x2="5.08" y2="30.226" width="0.6096" layer="1"/>
 <via x="5.08" y="29.718" extent="1-16" drill="0.6"/>
-<wire x1="5.08" y1="29.718" x2="7.874" y2="29.718" width="0.6096" layer="16"/>
-<wire x1="7.874" y1="29.718" x2="8.89" y2="30.734" width="0.6096" layer="16"/>
-<wire x1="5.08" y1="30.226" x2="5.08" y2="29.718" width="0.6096" layer="1"/>
-<wire x1="3" y1="37.432" x2="3" y2="31.798" width="0.6096" layer="1"/>
-<wire x1="3" y1="31.798" x2="5.08" y2="29.718" width="0.6096" layer="1"/>
 <wire x1="3" y1="4.732" x2="3" y2="10.112" width="0.6096" layer="1"/>
 <wire x1="3" y1="10.112" x2="4.59" y2="11.702" width="0.6096" layer="1"/>
@@
 <wire x1="17.48" y1="63.8" x2="17.272" y2="64.008" width="0.6096" layer="1"/>
 <wire x1="17.272" y1="64.008" x2="0.762" y2="64.008" width="0.6096" layer="1"/>
-<wire x1="17.48" y1="62.398" x2="13.884" y2="62.398" width="0.6096" layer="1"/>
-<wire x1="13.884" y1="62.398" x2="13.208" y2="61.722" width="0.6096" layer="1"/>
-<wire x1="13.208" y1="61.722" x2="13.208" y2="56.642" width="0.6096" layer="1"/>
-<wire x1="14.097" y1="55.753" x2="13.208" y2="56.642" width="0.6096" layer="1"/>
-<wire x1="15.74" y1="55.753" x2="14.097" y2="55.753" width="0.6096" layer="1"/>
-<wire x1="14.097" y1="55.753" x2="13.208" y2="54.864" width="0.6096" layer="1"/>
-<wire x1="13.208" y1="54.864" x2="13.208" y2="53.594" width="0.6096" layer="1"/>
-<wire x1="15.24" y1="53.213" x2="13.589" y2="53.213" width="0.6096" layer="1"/>
-<wire x1="13.589" y1="53.213" x2="13.208" y2="53.594" width="0.6096" layer="1"/>
 <wire x1="15.24" y1="53.213" x2="17.145" y2="53.213" width="0.6096" layer="1"/>
-<wire x1="17.145" y1="53.213" x2="17.78" y2="52.578" width="0.6096" layer="1"/>
+<wire x1="17.145" y1="53.213" x2="17.653" y2="52.705" width="0.6096" layer="1"/>
+<wire x1="17.653" y1="52.705" x2="17.78" y2="52.578" width="0.6096" layer="1"/>
 <wire x1="17.78" y1="52.578" x2="17.78" y2="47.498" width="0.6096" layer="1"/>
 <wire x1="17.78" y1="47.498" x2="17.78" y2="46.228" width="0.6096" layer="1"/>
 <wire x1="17.78" y1="46.228" x2="17.78" y2="45.212" width="0.6096" layer="1"/>
-<wire x1="17.78" y1="45.212" x2="17.78" y2="41.148" width="0.6096" layer="1"/>
+<wire x1="17.78" y1="45.212" x2="17.78" y2="39.116" width="0.6096" layer="1"/>
 <wire x1="15.24" y1="48.133" x2="17.145" y2="48.133" width="0.6096" layer="1"/>
 <wire x1="17.145" y1="48.133" x2="17.78" y2="47.498" width="0.6096" layer="1"/>
@@
 <wire x1="15.74" y1="45.593" x2="17.399" y2="45.593" width="0.6096" layer="1"/>
 <wire x1="17.399" y1="45.593" x2="17.78" y2="45.212" width="0.6096" layer="1"/>
-<wire x1="17.78" y1="41.148" x2="12.954" y2="36.322" width="0.6096" layer="1"/>
-<wire x1="12.954" y1="36.322" x2="12.954" y2="34.798" width="0.6096" layer="1"/>
 <wire x1="6.45" y1="19.322" x2="7.892" y2="19.322" width="0.6096" layer="1"/>
 <wire x1="7.892" y1="19.322" x2="8.128" y2="19.558" width="0.6096" layer="1"/>
-<wire x1="8.89" y1="30.734" x2="9.652" y2="30.734" width="0.6096" layer="16"/>
-<wire x1="9.652" y1="30.734" x2="11.176" y2="29.21" width="0.6096" layer="16"/>
 <wire x1="8.89" y1="26.416" x2="8.89" y2="30.734" width="0.6096" layer="1"/>
 <wire x1="8.128" y1="19.558" x2="8.128" y2="15.748" width="0.6096" layer="16"/>
@@
 <wire x1="8.636" y1="22.352" x2="8.636" y2="20.066" width="0.6096" layer="1"/>
 <wire x1="8.636" y1="20.066" x2="8.128" y2="19.558" width="0.6096" layer="1"/>
-<wire x1="8.526" y1="22.462" x2="6.6" y2="22.462" width="0.6096" layer="1"/>
-<wire x1="8.636" y1="22.352" x2="8.526" y2="22.462" width="0" layer="19" extent="1-1"/>
+<wire x1="5.08" y1="30.48" x2="11.938" y2="37.338" width="0.6096" layer="16"/>
+<wire x1="11.938" y1="37.338" x2="16.002" y2="37.338" width="0.6096" layer="16"/>
+<wire x1="16.002" y1="37.338" x2="17.78" y2="39.116" width="0.6096" layer="16"/>
+<via x="17.78" y="39.116" extent="1-16" drill="0.6"/>
+<wire x1="17.48" y1="62.398" x2="4.486" y2="62.398" width="0.6096" layer="1"/>
+<wire x1="3" y1="37.432" x2="3" y2="10.112" width="0.6096" layer="1"/>
+<wire x1="4.486" y1="62.398" x2="3" y2="60.912" width="0.6096" layer="1"/>
+<wire x1="3" y1="60.912" x2="3" y2="37.432" width="0.6096" layer="1"/>
+<wire x1="15.74" y1="55.753" x2="17.145" y2="55.753" width="0.6096" layer="1"/>
+<wire x1="17.145" y1="55.753" x2="17.78" y2="55.118" width="0.6096" layer="1"/>
+<wire x1="17.78" y1="55.118" x2="17.78" y2="52.832" width="0.6096" layer="1"/>
+<wire x1="17.78" y1="52.832" x2="17.653" y2="52.705" width="0.6096" layer="1"/>
+<wire x1="6.6" y1="22.462" x2="5.478" y2="22.462" width="0.6096" layer="1"/>
+<wire x1="5.478" y1="22.462" x2="4.826" y2="23.114" width="0.6096" layer="1"/>
+<wire x1="4.826" y1="23.114" x2="4.826" y2="29.464" width="0.6096" layer="1"/>
+<wire x1="4.826" y1="29.464" x2="5.08" y2="29.718" width="0.6096" layer="1"/>
+<wire x1="6.6" y1="22.462" x2="8.526" y2="22.462" width="0.6096" layer="1"/>
+<wire x1="8.526" y1="22.462" x2="8.636" y2="22.352" width="0.6096" layer="1"/>
+<wire x1="5.08" y1="30.226" x2="5.08" y2="29.718" width="0.6096" layer="1"/>
+<wire x1="5.08" y1="30.48" x2="5.08" y2="29.718" width="0.6096" layer="16"/>
 </signal>
 </signals>
